Commit message: Update arm.urdf.xacro

File: src/armando_description/urdf/arm.urdf.xacro (robot description, xacro)
@@ -34,4 +34,26 @@
     </inertial>
   </link>
+  <link name="camera_link">
+    <visual>
+      <geometry>
+        <box size="0.02 0.05 0.02"/>
+      </geometry>
+      <material name="white"/>
+    </visual>
+    <collision>
+      <geometry>
+        <box size="0.02 0.05 0.02"/>
+      </geometry>
+    </collision>
+    <inertial>
+      <mass value="0.01"/>
+      <inertia ixx="1e-6" ixy="0" ixz="0" iyy="1e-6" iyz="0" izz="1e-6"/>
+    </inertial>
+  </link>
+  <joint name="camera_joint" type="fixed">
+    <parent link="base_link"/>
+    <child link="camera_link"/>
+    <origin xyz="0.05 0 0.025" rpy="0 0 0"/>
+  </joint>
   <joint name="base_1_2" type="fixed">
     <parent link="base_link"/>
